File: KiCAD Files/EnergyMeter.kicad_pcb (KiCad board)
At the start: 2 copper layers, 50 parts, among them J2 Conn_01x05, Q1 BSS138, Q2 BSS138, Q3 S8050-SOT23, Q4 S8050-SOT23, SW1 SW_Push, U1 AMS1117-3.3, U2 ESP-12F, U3 HLW8032

Commit message: Layout
Parts:
- added J1: Screw_Terminal_AC, Library:KF7.62-2P, F.Cu at (90.8, 50.0)
- added J3: Screw_Terminal_LOAD, Library:KF7.62-2P, F.Cu at (89.2, 85.5)
- R6, R7: moved to B.Cu
- moved R13 167.0 mm to (96.5, 81.4), turned to 90 degrees
- moved R14 164.1 mm to (99.5, 81.4), turned to 90 degrees
- moved R11 163.5 mm to (97.6, 71.5)
- moved R10 163.5 mm to (97.9, 67.0)
- moved R15 161.2 mm to (102.4, 81.4), turned to 90 degrees
- moved R16 158.5 mm to (105.3, 81.4), turned to 90 degrees
- moved C11 154.6 mm to (102.0, 67.0)
- moved C12 154.4 mm to (102.0, 71.5)
- moved R12 152.6 mm to (110.9, 82.0)
- moved C10 148.8 mm to (107.5, 64.5)
- moved C13 144.2 mm to (111.0, 85.0), turned to 180 degrees
- moved C9 142.7 mm to (114.0, 64.5)
- moved R8 133.5 mm to (83.0, 69.5), turned to -90 degrees
- moved R6 131.3 mm to (83.0, 69.5), turned to -90 degrees
- moved R9 128.2 mm to (90.0, 69.5), turned to -90 degrees
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Connections:
- FL1 pad 1: Net-(C1-Pad1) -> Net-(PS1-AC/L)
- FL1 pad 2: Net-(PS1-AC/L) -> Net-(C1-Pad1)

Commit message: pcb layout
Parts:
- added H1: MountingHole, MountingHole:MountingHole_3.2mm_M3, F.Cu at (74.5, 28.0)
- added H2: MountingHole, MountingHole:MountingHole_3.2mm_M3, F.Cu at (167.5, 28.0)
- added H3: MountingHole, MountingHole:MountingHole_3.2mm_M3, F.Cu at (167.5, 113.0)
- added H4: MountingHole, MountingHole:MountingHole_3.2mm_M3, F.Cu at (74.5, 113.0)
- U3: footprint Package_SO:SOP-8_3.9x4.9mm_P1.27mm -> Library:SOP-8_3.9x4.9mm_P1.27mm_custom
- moved D1 177.0 mm to (112.0, 95.9), turned to 90 degrees
- moved R1 161.7 mm to (112.0, 91.9), turned to -90 degrees
- moved R21 156.4 mm to (125.0, 104.1), turned to -90 degrees
- moved C6 153.7 mm to (116.0, 94.0), turned to -90 degrees
- moved C5 152.4 mm to (120.0, 94.0), turned to -90 degrees
- moved C7 140.9 mm to (138.0, 84.0), turned to -90 degrees
- moved R22 140.6 mm to (142.5, 100.9), turned to 90 degrees
- moved C4 135.0 mm to (134.5, 94.0), turned to -90 degrees
- moved C3 134.3 mm to (138.5, 94.0), turned to -90 degrees
- moved C8 131.6 mm to (143.0, 84.5), turned to -90 degrees
- moved J2 131.6 mm to (141.1, 106.1), turned to -90 degrees
- moved R5 127.0 mm to (158.0, 78.4), turned to -90 degrees
- moved SW1 122.8 mm to (159.5, 71.0), turned to 180 degrees
- moved R2 122.7 mm to (150.0, 104.0), turned to -90 degrees
- moved R3 120.7 mm to (162.0, 78.5), turned to -90 degrees
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Connections:
- J3 pad 1: Net-(J3-Pin_1) -> L
- J3 pad 2: L -> Net-(J3-Pin_2)
- R11 pad 1: Net-(J3-Pin_1) -> Net-(J3-Pin_2)
- R6 pad 2: Net-(J3-Pin_1) -> Net-(J3-Pin_2)
- R7 pad 2: Net-(J3-Pin_1) -> Net-(J3-Pin_2)
- R8 pad 2: Net-(J3-Pin_1) -> Net-(J3-Pin_2)
- R9 pad 2: Net-(J3-Pin_1) -> Net-(J3-Pin_2)
Routing:
- net L: track 0.00 -> 99.4 mm
- net N: track 0.00 -> 82.5 mm
- net Net-(J3-Pin_2): track 0.00 -> 63.2 mm
- net +5V: track 0.00 -> 55.1 mm
- net Net-(C1-Pad1): track 0.00 -> 40.8 mm
- net Net-(PS1-AC/L): track 0.00 -> 37.6 mm
- net Net-(PS1-AC/N): track 0.00 -> 28.6 mm
- net Net-(U3-VP): track 0.00 -> 16.2 mm
- net Net-(U3-IP): track 0.00 -> 12.7 mm
- net Net-(U3-IN): track 0.00 -> 12.0 mm
- net Net-(R15-Pad2): track 0.00 -> 2.17 mm
- net Net-(R14-Pad2): track 0.00 -> 2.17 mm
- net Net-(R13-Pad2): track 0.00 -> 2.17 mm
Other:
- board outline added: 100 x 92 mm
- board text added: "DTR"
- board text added: "GND"
- board text added: "RTS"
- board text added: "RX"
- board text added: "TX"

Commit message: V1rev1
Parts:
- H1, H2, H3, H4: footprint MountingHole:MountingHole_3.2mm_M3 -> MountingHole:MountingHole_3.2mm_M3_Pad_TopBottom
- moved R20 137.7 mm to (146.0, 93.2), turned to -90 degrees
- moved R18 136.5 mm to (146.0, 97.9), turned to -90 degrees
- moved JP1 132.8 mm to (151.8, 110.5), turned to 180 degrees
- moved R19 128.2 mm to (155.0, 93.2), turned to 90 degrees
- moved R17 127.0 mm to (155.0, 98.0), turned to 90 degrees
- moved Q2 95.3 mm to (150.4, 93.2), turned to 180 degrees
- moved Q1 90.7 mm to (150.4, 98.0), turned to 180 degrees
- moved R1 80.1 mm to (189.2, 113.1), turned to 90 degrees
- moved D1 78.4 mm to (189.2, 109.1), turned to -90 degrees
- moved C6 63.6 mm to (179.5, 89.7), turned to 90 degrees
- moved C5 57.2 mm to (177.0, 89.7), turned to 90 degrees
- moved SW1 54.4 mm to (186.0, 118.6), turned to 0 degrees
- moved C2 50.7 mm to (186.5, 84.3), turned to -90 degrees
- moved U1 43.6 mm to (171.0, 89.7), turned to 0 degrees
- moved R3 40.9 mm to (183.8, 113.2), turned to 180 degrees
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Routing:
- net +3.3V: track 0.00 -> 132.2 mm, vias 0 -> 2
- net L: track 99.4 -> 19.3 mm
- net RESET: track 0.00 -> 71.9 mm, vias 0 -> 4
- net Net-(J3-Pin_2): track 63.2 -> 5.09 mm
- net +5V: track 55.1 -> 105.5 mm, vias 0 -> 2
- net N: track 82.5 -> 32.1 mm
- net PF: track 0.00 -> 39.4 mm, vias 0 -> 2
- net Net-(PS1-AC/L): track 37.6 -> 8.91 mm
- net TX: track 0.00 -> 26.0 mm
- net GPIO0: track 0.00 -> 25.3 mm, vias 0 -> 4
- net /RTS: track 0.00 -> 23.9 mm
- net Net-(JP1-B): track 0.00 -> 19.0 mm
- net Net-(PS1-AC/N): track 28.6 -> 10.1 mm
- net RX: track 0.00 -> 12.9 mm
- net Net-(U2-EN): track 0.00 -> 11.0 mm
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- added copper zone on B.Cu, net GND
- added copper zone on F.Cu, net GND
- added copper zone on B.Cu, net L
- added copper zone on F.Cu, net L
- added copper zone on B.Cu, net N
- added copper zone on F.Cu, net N
- added copper zone on B.Cu, net Net-(J3-Pin_2)
- added copper zone on F.Cu, net Net-(J3-Pin_2)
Other:
- board size 100 x 92 mm -> 94 x 82 mm
- board text added: "230VAC"
- board text added: "EnergyMeterV1rev1"
- board text added: "JLCJLCJLCJLC"
- board text added: "LOAD"
- board text added: "POWER"
- board text added: "RESET"

Commit message: update
Parts:
- F1: value 500mA, SLOW, socketed -> Fuse socket
Connections:
- H1 pad 1: (no net) -> unconnected-(H1-Pad1)
- H2 pad 1: (no net) -> unconnected-(H2-Pad1)_2
- H3 pad 1: (no net) -> unconnected-(H3-Pad1)_2
- H4 pad 1: (no net) -> unconnected-(H4-Pad1)_2
Routing:
- net GND: vias 18 -> 43
