File: KiCAD Files/EnergyMeter.kicad_pcb (KiCad board)
At the start: 2 copper layers, 94 x 82 mm, 56 parts, among them J1 Screw_Terminal_AC, J2 Conn_01x05, J3 Screw_Terminal_LOAD, Q1 BSS138, Q2 BSS138, Q3 S8050-SOT23, Q4 S8050-SOT23, SW1 SW_Push, U1 AMS1117-3.3, U2 ESP-12F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

Commit message: update
Parts:
- removed JP1: Jumper_2_Bridged, Connector_PinHeader_2.54mm:PinHeader_1x02_P2.54mm_Vertical
- removed Q1, Q2: BSS138, Package_TO_SOT_SMD:SOT-23
- added C14: 100u, Capacitor_SMD:C_Elec_10x10.2, F.Cu at (247.8, 98.0)
- added C15: 100n, Capacitor_SMD:C_0805_2012Metric, F.Cu at (220.2, 115.7)
- added C16: 100n, Capacitor_SMD:C_0805_2012Metric, F.Cu at (220.2, 118.7)
- added C17: 10u, Capacitor_SMD:C_1206_3216Metric, F.Cu at (251.8, 76.6)
- added C18: 10u, Capacitor_SMD:C_1206_3216Metric, F.Cu at (251.8, 79.9)
- added D2: MB6S, Package_TO_SOT_SMD:TO-269AA, F.Cu at (152.5, 96.0)
- added D3: US1JHE3, Diode_SMD:D_SMA, F.Cu at (233.5, 107.8)
- added D4: US1JHE3, Diode_SMD:D_SMA, F.Cu at (233.5, 112.3)
- added L1: 1mH, Inductor_SMD:L_Taiyo-Yuden_NR-80xx_HandSoldering, F.Cu at (223.7, 96.8)
- added L2: 1mH, Inductor_SMD:L_Taiyo-Yuden_NR-80xx_HandSoldering, F.Cu at (223.7, 106.4)
- added R23: 470R, Resistor_SMD:R_0805_2012Metric, F.Cu at (246.7, 81.2)
- added R24: 10k, Resistor_SMD:R_0805_2012Metric, F.Cu at (246.7, 84.2)
- added R25: 3k3, Resistor_SMD:R_0805_2012Metric, F.Cu at (246.7, 87.1)
- added SW2: SW_SPST, Button_Switch_SMD:SW_DIP_SPSTx01_Slide_6.7x4.1mm_W6.73mm_P2.54mm_LowProfile_JPin, F.Cu at (234.7, 117.5)
- added TP1: TestPoint, TestPoint:TestPoint_Pad_D3.0mm, F.Cu at (255.0, 106.5)
- added TP2: TestPoint, TestPoint:TestPoint_Pad_D3.0mm, F.Cu at (255.0, 111.5)
- added U4: PC817, Package_DIP:DIP-4_W7.62mm, F.Cu at (231.1, 94.2)
- added U5: PC817, Package_DIP:DIP-4_W7.62mm, F.Cu at (231.1, 100.8)
- added U6: AMS1117-5.0, Package_TO_SOT_SMD:SOT-223-3_TabPin2, F.Cu at (211.0, 116.0)
- C2: value 100u -> 100uF
- C3: value 10u -> 4u7 / 400V; footprint Capacitor_SMD:C_1206_3216Metric -> Capacitor_SMD:CP_Elec_8x10
- C4: value 100n -> 4u7 / 400V; footprint Capacitor_SMD:C_0805_2012Metric -> Capacitor_SMD:CP_Elec_8x10
- C5: value 10u -> 100n; footprint Capacitor_SMD:C_1206_3216Metric -> Capacitor_SMD:C_0805_2012Metric
- C6: value 100n -> 22u / 50V; footprint Capacitor_SMD:C_0805_2012Metric -> Capacitor_SMD:C_2220_5750Metric_Pad1.97x5.40mm_HandSolder
- J2: footprint Connector_PinHeader_2.54mm:PinHeader_1x05_P2.54mm_Horizontal -> Connector_PinHeader_2.54mm:PinHeader_1x05_P2.54mm_Vertical
- PS1: value HLK-PM01 -> HLK-PM03
- R17: value 10k -> 470R
- R19: value 10k -> 2k05
- R20: value 10k -> 13k
- U1: value AMS1117-3.3 -> LNK304G; footprint Package_TO_SOT_SMD:SOT-223-3_TabPin2 -> Package_DIP:PowerIntegrations_SMD-8B
- moved R18 103.9 mm to (246.7, 72.4), turned to 0 degrees
- moved R20 101.8 mm to (246.7, 78.3), turned to 0 degrees
- moved R17 96.1 mm to (246.7, 69.4), turned to 0 degrees
- moved R19 93.5 mm to (246.7, 75.3), turned to 0 degrees
- moved U1 78.0 mm to (246.4, 109.8)
- moved C6 76.1 mm to (253.3, 71.4), turned to 0 degrees
- moved C3 50.2 mm to (212.2, 97.0), turned to 0 degrees
- moved C4 50.2 mm to (212.2, 106.8), turned to 0 degrees
- moved C5 48.9 mm to (220.2, 112.7), turned to 0 degrees
- moved J2 42.0 mm to (189.0, 104.1), turned to 180 degrees
- moved F1 4.41 mm to (120.8, 57.0)
- moved PS1 3.05 mm to (154.5, 67.0)
- moved FL1 2.25 mm to (143.4, 73.0)
- moved C1 1.50 mm to (132.1, 65.5)
- moved RV1 0.75 mm to (124.8, 69.2)
Connections:
- net Net-(PS1-AC/L) renamed /L_COMM
- net Net-(PS1-AC/N) renamed /N_COMM
- C10 pad 2: GND -> GND1
- C11 pad 2: GND -> GND1
- C12 pad 2: GND -> GND1
- C13 pad 2: GND -> GND1
- C2 pad 1: +5V -> +3.3V
- C2 pad 2: GND -> GND2
- C3 pad 1: +5V -> Net-(D2-+)
- C3 pad 2: GND -> GND1
- C4 pad 1: +5V -> Net-(U1-D)
- C4 pad 2: GND -> GND1
- C5 pad 1: +3.3V -> Net-(U1-BP)
- C5 pad 2: GND -> Net-(D3-K)
- C6 pad 1: +3.3V -> Net-(D4-K)
- C6 pad 2: GND -> Net-(D3-K)
- C7 pad 2: GND -> GND2
- C8 pad 2: GND -> GND2
- C9 pad 2: GND -> GND1
- D1 pad 1: GND -> GND2
- J2 pad 5: GND -> GND2
- PS1 pad 3: GND -> GND2
- PS1 pad 4: +5V -> +3.3V
- R12 pad 1: GND -> GND1
- R17 pad 1: +3.3V -> +5V
- R18 pad 1: +5V -> +3.3V
- R18 pad 2: HLW8032 TX -> PF
- R19 pad 1: +3.3V -> Net-(U1-FB)
- R19 pad 2: PF -> Net-(D3-K)
- R2 pad 2: GND -> GND2
- R20 pad 1: +5V -> Net-(U1-FB)
- R20 pad 2: HLW8032 PF -> Net-(D4-K)
- SW1 pad 2: GND -> GND2
- U1 pad 1: GND -> Net-(D3-K)
- U1 pad 2: +3.3V -> Net-(D3-K)
- U1 pad 3: +5V -> Net-(U1-BP)
- U2 pad 15: GND -> GND2
- U3 pad 5: GND -> GND1
Routing:
- net +3.3V: track 132.2 -> 0.00 mm, vias 2 -> 0
- net +5V: track 105.5 -> 0.00 mm, vias 2 -> 0
- net RESET: track 71.9 -> 0.00 mm, vias 4 -> 0
- net PF: track 39.4 -> 0.00 mm, vias 2 -> 0
- net Net-(C1-Pad1): track 38.7 -> 0.00 mm
- net N: track 32.1 -> 0.00 mm
- net TX: track 26.0 -> 0.00 mm
- net GPIO0: track 25.3 -> 0.00 mm, vias 4 -> 0
- net /RTS: track 23.9 -> 0.00 mm
- net L: track 19.3 -> 0.00 mm
- net Net-(R17-Pad2): track 19.0 -> 0.00 mm
- net Net-(U3-IP): track 15.2 -> 0.00 mm
- net Net-(U3-VP): track 14.6 -> 0.00 mm
- net Net-(U3-IN): track 13.2 -> 0.00 mm
- net RX: track 12.9 -> 0.00 mm
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- removed copper zone on B.Cu, net GND
- removed copper zone on F.Cu, net GND
Other:
- board text added: "EnergyMeterV1rev2"
- board text removed: "EnergyMeterV1rev1"

Commit message: Update EnergyMeter.kicad_pcb
Parts:
- moved D4 87.5 mm to (248.0, 26.0)
- moved L2 82.5 mm to (256.2, 30.6), turned to 90 degrees
- moved U1 81.3 mm to (227.2, 30.8), turned to 180 degrees
- moved C5 80.5 mm to (235.5, 33.6), turned to -90 degrees
- moved R21 78.2 mm to (215.1, 84.0)
- moved R22 78.2 mm to (215.1, 74.9)
- moved Q3 78.2 mm to (212.5, 79.4)
- moved Q4 78.2 mm to (217.5, 79.4)
- moved L1 77.2 mm to (210.5, 20.8)
- moved C4 75.2 mm to (215.5, 31.8), turned to -90 degrees
- moved D2 74.9 mm to (191.5, 32.0), turned to 0 degrees
- moved D3 71.8 mm to (242.2, 36.5), turned to -90 degrees
- moved C14 66.6 mm to (266.5, 34.1), turned to -90 degrees
- moved C3 65.6 mm to (205.0, 31.8), turned to -90 degrees
- moved H1 57.0 mm to (102.0, 110.0)
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Routing:
- removed copper zone on B.Cu, net L
- removed copper zone on F.Cu, net L
- removed copper zone on B.Cu, net N
- removed copper zone on F.Cu, net N
- removed copper zone on B.Cu, net Net-(J3-Pin_2)
- removed copper zone on F.Cu, net Net-(J3-Pin_2)
Other:
- outline, holes or cut-outs redrawn
