File: KiCAD Files/EnergyMeter.kicad_sch (KiCad schematic)
At the start: 56 parts, among them J1 Screw_Terminal_AC, J2 Conn_01x05, J3 Screw_Terminal_LOAD, Q1 BSS138, Q2 BSS138, Q3 S8050-SOT23, Q4 S8050-SOT23, SW1 SW_Push, U1 AMS1117-3.3, U2 ESP-12F, U3 HLW8032

Commit message: V1rev1
Parts:
- H1, H2, H3, H4: footprint MountingHole:MountingHole_3.2mm_M3 -> MountingHole:MountingHole_3.2mm_M3_Pad_TopBottom
Changed lines of the file:
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@@
 			)
 		)
-		(property "Footprint" "MountingHole:MountingHole_3.2mm_M3"
+		(property "Footprint" "MountingHole:MountingHole_3.2mm_M3_Pad_TopBottom"
 			(at 99.06 185.42 0)
 			(effects
@@
 			)
 		)
-		(property "Footprint" "MountingHole:MountingHole_3.2mm_M3"
+		(property "Footprint" "MountingHole:MountingHole_3.2mm_M3_Pad_TopBottom"
 			(at 137.16 185.42 0)
 			(effects
@@
 			)
 		)
-		(property "Footprint" "MountingHole:MountingHole_3.2mm_M3"
+		(property "Footprint" "MountingHole:MountingHole_3.2mm_M3_Pad_TopBottom"
 			(at 118.11 185.42 0)
 			(effects
@@
 			)
 		)
-		(property "Footprint" "MountingHole:MountingHole_3.2mm_M3"
+		(property "Footprint" "MountingHole:MountingHole_3.2mm_M3_Pad_TopBottom"
 			(at 80.01 185.42 0)
 			(effects

Commit message: update
Other:
- note added: "TO-DO: - BOM needs to include both the fuse and fuse socket - BOM needs to include jumper - add every datasheet link to BOM"
- note removed: "TO-DO: - galvanski odvojiti signale - provjeriti pinout od choke - BOM needs to include both the fuse and fuse socket - BOM needs to include jumper - add every datasheet link to BOM - vidjeti što imam od ovih komponenata"
Changed lines of the file:
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@@
 		)
 	)
-	(text "TO-DO:\n- galvanski odvojiti signale\n- provjeriti pinout od choke\n- BOM needs to include both the fuse and fuse socket\n- BOM needs to include jumper\n- add every datasheet link to BOM\n- vidjeti što imam od ovih komponenata\n"
+	(text "TO-DO:\n- BOM needs to include both the fuse and fuse socket\n- BOM needs to include jumper\n- add every datasheet link to BOM\n"
 		(exclude_from_sim no)
 		(at 227.33 153.162 0)

Commit message: update
Other:
- note added: "TO-DO: - BOM needs to include both the fuse and fuse socket - BOM needs to include jumper - add every datasheet link to BOM - github documentation - kućište"
- note removed: "TO-DO: - BOM needs to include both the fuse and fuse socket - BOM needs to include jumper - add every datasheet link to BOM"
Changed lines of the file:
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@@
 		)
 	)
-	(text "TO-DO:\n- BOM needs to include both the fuse and fuse socket\n- BOM needs to include jumper\n- add every datasheet link to BOM\n"
+	(text "TO-DO:\n- BOM needs to include both the fuse and fuse socket\n- BOM needs to include jumper\n- add every datasheet link to BOM\n- github documentation\n- kućište"
 		(exclude_from_sim no)
 		(at 227.33 153.162 0)

Commit message: update
Parts:
- added F2: 500mA, SLOW, symbol Device:Fuse_Small
- added JP2: ~, symbol Symbol_Library:Jumper
- F1: value 500mA, SLOW, socketed -> Fuse socket
- H1, H2, H3, H4: symbol Mechanical:MountingHole -> Mechanical:MountingHole_Pad
Connections:
- no-connect marks 13 -> 19
Other:
- note added: "TO-DO: - github documentation - kućište"
- note removed: "TO-DO: - BOM needs to include both the fuse and fuse socket - BOM needs to include jumper - add every datasheet link to BOM - github documentation - kućište"

Commit message: update
Other:
- note removed: "TO-DO: - github documentation - kućište"
Changed lines of the file:
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@@
-		)
-	)
-	(text "TO-DO:\n- github documentation\n- kućište"
-		(exclude_from_sim no)
-		(at 257.81 161.798 0)
-		(effects
-			(font
-				(size 1.27 1.27)
-			)
-			(justify left)
 		)
 	)

Commit message: Update EnergyMeter.kicad_sch
Other:
- note added: "TO-DO: - sklopka umjesto jumpera - Galvanski odvojiti GNDove (dodati optocouplere) - Pinovi serijske kom. i PF-a za debugiranje - relej? - ulaz za temp. senzor?"
Changed lines of the file:
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@@
+		)
+	)
+	(text "TO-DO:\n- sklopka umjesto jumpera\n- Galvanski odvojiti GNDove (dodati optocouplere)\n- Pinovi serijske kom. i PF-a za debugiranje\n- relej?\n- ulaz za temp. senzor?"
+		(exclude_from_sim no)
+		(at 192.786 145.288 0)
+		(effects
+			(font
+				(size 1.27 1.27)
+			)
+			(justify left)
 		)
 	)

Commit message: Update EnergyMeter.kicad_sch
Other:
- note added: "TO-DO: - sklopka umjesto jumpera - Galvanski odvojiti GNDove/napajanja - Dodati optocouplere - Maknuti LogicLevelConverter - Pinovi serijske kom. i PF-a za debugiranje - relej? - ulaz za temp. senzor?"
- note removed: "TO-DO: - sklopka umjesto jumpera - Galvanski odvojiti GNDove (dodati optocouplere) - Pinovi serijske kom. i PF-a za debugiranje - relej? - ulaz za temp. senzor?"
Changed lines of the file:
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@@
 		)
 	)
-	(text "TO-DO:\n- sklopka umjesto jumpera\n- Galvanski odvojiti GNDove (dodati optocouplere)\n- Pinovi serijske kom. i PF-a za debugiranje\n- relej?\n- ulaz za temp. senzor?"
+	(text "TO-DO:\n- sklopka umjesto jumpera\n- Galvanski odvojiti GNDove/napajanja\n- Dodati optocouplere\n- Maknuti LogicLevelConverter\n- Pinovi serijske kom. i PF-a za debugiranje\n- relej?\n- ulaz za temp. senzor?"
 		(exclude_from_sim no)
 		(at 192.786 145.288 0)

Commit message: update
Parts:
- removed JP1: Jumper_2_Bridged, Connector_PinHeader_2.54mm:PinHeader_1x02_P2.54mm_Vertical, symbol Jumper:Jumper_2_Bridged
- removed JP2: ~, symbol Symbol_Library:Jumper
- removed Q1, Q2: BSS138, Package_TO_SOT_SMD:SOT-23, symbol Transistor_FET:BSS138
- removed R19, R20: 10k, Resistor_SMD:R_0805_2012Metric, symbol Device:R_Small
- added C14: 47u, symbol Device:C_Polarized_Small
- added R23: 470R, Resistor_SMD:R_0805_2012Metric, symbol Device:R_Small
- added R24: 10k, Resistor_SMD:R_0805_2012Metric, symbol Device:R_Small
- added SW2: SW_SPST, symbol Switch:SW_SPST
- added U4, U5: PC817, Package_DIP:DIP-4_W7.62mm, symbol Isolator:PC817
- added U6: LR8N8-G, Package_TO_SOT_SMD:SOT-89-3, symbol Regulator_Linear:LR8N8-G
- R17: value 10k -> 470R; LCSC Part # C105877 -> C95781
- R18: LCSC Part # C105877 -> C95781
Connections:
- net +3.3V: now also R18.1, R24.1; no longer R17.1
- net +5V: now also R17.1, R23.1; no longer R18.1
- net GND: no longer C2.2, C3.2, C4.2, C5.2, C6.2, C7.2, C8.2, D1.1 (K), J2.5 (Pin_5), PS1.3 (-Vout), R2.2, SW1.2, U1.1 (GND), U2.15 (GND)
- net HLW8032 PF: now also U5.2
- net HLW8032 TX: now also U4.2; no longer R18.2
- net PF: now also R18.2, U5.4
- net TX: now also SW2.2 (B)
- net at R17.2: now also U5.1
- net L_COM: now reaches FL1.1, PS1.1 (AC/L)
- net N_COM: now reaches FL1.4, PS1.2 (AC/N)
- new net: R24.2, SW2.1 (A), U4.4
- new net: R23.2, U4.1
- new net: C14.1, U6.1 (IN)
- new net GND1: C14.2
- new net GND2: C2.2, C3.2, C4.2, C5.2, C6.2, C7.2, C8.2, D1.1 (K), J2.5 (Pin_5), PS1.3 (-Vout), R2.2, SW1.2, U1.1 (GND), U2.15 (GND), U4.3, U5.3
Other:
- note added: "OPTO-ISOLATORS"
- note added: "TO-DO: - MP150 5V/200mA za napajanje senzora, na ulazu ispraviti napon - Maknuti LogicLevelConverter - Pinovi serijske kom. i PF-a za debugiranje (iza optocouplera) - relej? - ulaz za temp. senzor? - paziti na GND-ove, N treba biti spojen na GND od senzora - PC817 SMD footprint? ako ih imam u labosu - sklopka footprint - C14 vrijednost i footprint?"
- note added: "The power supply of the HLW8032 chip should be non-isolated"
- note removed: "LOGIC LEVEL CONVERSION"
- note removed: "TO-DO: - sklopka umjesto jumpera - Galvanski odvojiti GNDove/napajanja - Dodati optocouplere - Maknuti LogicLevelConverter - Pinovi serijske kom. i PF-a za debugiranje - relej? - ulaz za temp. senzor?"
- moved on the sheet: C2, PS1
