File: KiCAD Files/EnergyMeter.kicad_sch (KiCad schematic)
At the start: 59 parts, among them J1 Screw_Terminal_AC, J2 Conn_01x05, J3 Screw_Terminal_LOAD, Q3 S8050-SOT23, Q4 S8050-SOT23, SW1 SW_Push, SW2 SW_SPST, U1 AMS1117-3.3, U2 ESP-12F, U3 HLW8032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

Commit message: Update EnergyMeter.kicad_sch
Parts:
- removed C3: 10u, Capacitor_SMD:C_1206_3216Metric, symbol Device:C_Small
- removed C4: 100n, Capacitor_SMD:C_0805_2012Metric, symbol Device:C_Small
- removed PS1: HLK-PM01, Converter_ACDC:Converter_ACDC_Hi-Link_HLK-PMxx, symbol Converter_ACDC:HLK-PM01
- removed U1: AMS1117-3.3, Package_TO_SOT_SMD:SOT-223-3_TabPin2, symbol Regulator_Linear:AMS1117-3.3
- removed U6: LR8N8-G, Package_TO_SOT_SMD:SOT-89-3, symbol Regulator_Linear:LR8N8-G
- added C15, C16: 100n, Capacitor_SMD:C_0805_2012Metric, symbol Device:C_Small
- added C17, C18: 10u, Capacitor_SMD:C_0805_2012Metric, symbol Device:C_Small
- added C3, C4: 4u7 / 400V, symbol Device:C_Polarized_Small
- added D2: MB6S, Package_TO_SOT_SMD:TO-269AA, symbol Diode_Bridge:MB6S
- added D3: UF4005, symbol Device:D_Small
- added D4: 1N4005GP, symbol Device:D_Small
- added L1, L2: 1mH, symbol Device:L_Small
- added PS1: HLK-PM03, Converter_ACDC:Converter_ACDC_Hi-Link_HLK-PMxx, symbol Converter_ACDC:HLK-PM03
- added R19: 2k05, Resistor_SMD:R_0805_2012Metric, symbol Device:R_Small
- added R20: 13k, Resistor_SMD:R_0805_2012Metric, symbol Device:R_Small
- added R25: 3k3, Resistor_SMD:R_0805_2012Metric, symbol Device:R_Small
- added TP1, TP2: TestPoint, symbol Connector:TestPoint
- added U1: LNK304P, Package_DIP:PowerIntegrations_PDIP-8B, symbol Regulator_Switching:LNK304P
- added U6: AMS1117-5.0, Package_TO_SOT_SMD:SOT-223-3_TabPin2, symbol Regulator_Linear:AMS1117-5.0
- C14: value 47u -> 100u
- C5: value 10u -> 100n; footprint Capacitor_SMD:C_1206_3216Metric -> (none); LCSC Part # C2174822 -> (none)
- C6: value 100n -> 10u / 50V; footprint Capacitor_SMD:C_0805_2012Metric -> (none); LCSC Part # C599848 -> (none)
Connections:
- net GND is gone; now on net GND1: C10.2, C11.2, C12.2, C13.2, C9.2, R12.1, U3.5 (GND)
- net +3.3V: now also C2.1, PS1.4 (+Vout); no longer C5.1, C6.1
- net +5V: now also C15.1, C18.1, U6.2 (VO); no longer C2.1
- net GND1: now also C15.2, C16.2, C17.2, C18.2, C3.2, C4.2, D2.4 (-), D3.2 (A), R25.2, U6.1 (GND)
- net GND2: now also PS1.3 (-Vout); no longer C5.2, C6.2
- net PF: now also TP2.1
- net at R24.2, SW2.1 (A), U4.4: now also TP1.1
- net +12V: now reaches C14.1
- net +12V: now also C16.1, C17.1, D4.2 (A), L2.2, R25.1, U6.3 (VI)
- net L_COM renamed L_COMM
- net L_COMM: now also D2.2, PS1.1 (AC/L)
- net N_COM renamed N_COMM
- net N_COMM: now also D2.1, PS1.2 (AC/N)
- new net: R19.1, R20.1, U1.4 (FB)
- new net: C6.1, D4.1 (K), R20.2
- new net: C5.1, U1.3 (BP)
- new net: C5.2, C6.2, D3.1 (K), L2.1, R19.2, U1.1 (S), U1.2 (S), U1.7 (S), U1.8 (S)
- new net: C3.1, D2.3 (+), L1.1
- new net: C4.1, L1.2, U1.5 (D)
Other:
- note added: "12V 120mA output"
- note added: "230VAC >> 3.3VDC"
- note added: "Non-isolated power supply for HLW8032 IC."
- note added: "TO-DO: - LNK304 non-isolating PSU - paziti na GND-ove, N treba biti spojen na GND od senzora - LCSC part # koji nedostaju - PC817 THT footprint - sklopka footprint - test point footprinti - provjeriti footprinte"
- note removed: "230VAC >> 5VDC"
- note removed: "5VDC >> 3.3VDC"
- note removed: "TO-DO: - MP150 5V/200mA za napajanje senzora, na ulazu ispraviti napon - Maknuti LogicLevelConverter - Pinovi serijske kom. i PF-a za debugiranje (iza optocouplera) - relej? - ulaz za temp. senzor? - paziti na GND-ove, N treba biti spojen na GND od senzora - PC817 SMD footprint? ako ih imam u labosu - sklopka footprint - C14 vrijednost i footprint?"
- note removed: "The power supply of the HLW8032 chip should be non-isolated"
- moved on the sheet: C1, C2, C7, C8, D1, F1, F2, FL1, J1, R1, R2, R3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

Commit message: update
Parts:
- removed U1: LNK304P, Package_DIP:PowerIntegrations_PDIP-8B, symbol Regulator_Switching:LNK304P
- added U1: LNK304G, Package_DIP:PowerIntegrations_SMD-8B, symbol Regulator_Switching:LNK304G
- C14: footprint (none) -> Capacitor_SMD:C_Elec_10x10.2; LCSC Part # (none) -> C5158069
- C17, C18: footprint Capacitor_SMD:C_0805_2012Metric -> Capacitor_SMD:C_1206_3216Metric; LCSC Part # C599848 -> C2174822
- C2: value 100u -> 100uF
- C3, C4: footprint (none) -> Capacitor_SMD:CP_Elec_8x10; LCSC Part # (none) -> C250872
- C5: footprint (none) -> Capacitor_SMD:C_0805_2012Metric; LCSC Part # (none) -> C599848
- C6: value 10u / 50V -> 22u / 50V; footprint (none) -> Capacitor_SMD:C_2220_5750Metric_Pad1.97x5.40mm_HandSolder; LCSC Part # (none) -> C784103
- D3: value UF4005 -> US1JHE3; footprint (none) -> Diode_SMD:D_SMA; LCSC Part # (none) -> C142585
- D4: value 1N4005GP -> US1JHE3; footprint (none) -> Diode_SMD:D_SMA; LCSC Part # (none) -> C142585
- J2: footprint Connector_PinHeader_2.54mm:PinHeader_1x05_P2.54mm_Horizontal -> Connector_PinHeader_2.54mm:PinHeader_1x05_P2.54mm_Vertical
- L1, L2: footprint (none) -> Inductor_SMD:L_Taiyo-Yuden_NR-80xx_HandSoldering; LCSC Part # (none) -> C19190456
- R18, R24: LCSC Part # C95781 -> C105877
- R19: LCSC Part # C105877 -> C2091315
- R20: LCSC Part # C105877 -> C137592
- R25: LCSC Part # C105877 -> C844842
- SW2: footprint (none) -> Button_Switch_SMD:SW_DIP_SPSTx01_Slide_6.7x4.1mm_W6.73mm_P2.54mm_LowProfile_JPin; LCSC Part # (none) -> C54948
- TP1, TP2: footprint (none) -> TestPoint:TestPoint_Pad_D3.0mm; now left out of the parts list
- U4, U5: LCSC Part # (none) -> C2833075
- U6: LCSC Part # (none) -> C22459281
Connections:
- net at R19.1, R20.1: now also U1.4 (FB)
- net at C5.1: now also U1.3 (BP)
- net at C5.2, C6.2, D3.1 (K)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: now also U1.1 (S), U1.2 (S), U1.7 (S), U1.8 (S)
- net at C4.1, L1.2: now also U1.5 (D)
Other:
- note removed: "TO-DO: - LNK304 non-isolating PSU - paziti na GND-ove, N treba biti spojen na GND od senzora - LCSC part # koji nedostaju - PC817 THT footprint - sklopka footprint - test point footprinti - provjeriti footprinte"
